File: Flaps&Spedd.kicad_pcb (KiCad board)
At the start: 2 copper layers, 46 x 46 mm, 22 parts, among them J1 CAN-M, J2 CAN-F, U1 SN65HVD230

Commit message: Fix: - Löcher Kontakte zu klein - DC Wandler Vin (12V) und Vout (5V) vertauscht - DC Wandler mehr zu Mitte - Widerstände und Kondensator anders Format
Parts:
- H1, H10, H11, H12, H13, H14, H2, H3, H4, H7, H8, H9: footprint Connector_PinHeader_1.27mm:PinHeader_1x01_P1.27mm_Vertical -> Connector_Pin:Pin_D0.9mm_L10.0mm_W2.4mm_FlatFork
- moved H4 10.2 mm to (73.6, 76.2)
- moved H1 5.12 mm to (66.0, 76.2)
- moved H2 2.80 mm to (71.0, 76.2)
- moved H3 2.80 mm to (68.5, 76.2)
Routing:
- net +12V: track 45.9 -> 32.3 mm, vias 2 -> 1
- net Net-(H1-Pad1): track 17.0 -> 12.5 mm
- net GND: track 81.0 -> 76.7 mm
- net Net-(JP1-B): track 17.8 -> 13.7 mm, vias 0 -> 2
- net +3V3: track 22.1 -> 18.3 mm
- net Net-(U1-Rs): track 4.91 -> 3.63 mm
