File: Flaps&Spedd.kicad_pcb (KiCad board)
At the start: 2 copper layers, 46 x 46 mm, 22 parts, among them J1 CAN-M, J2 CAN-F, U1 SN65HVD230

Commit message: Fix: - Löcher Kontakte zu klein - DC Wandler Vin (12V) und Vout (5V) vertauscht - DC Wandler mehr zu Mitte - Widerstände und Kondensator anders Format
Parts:
- C1: footprint Capacitor_SMD:C_0201_0603Metric -> Connector_PinHeader_1.00mm:PinHeader_1x01_P1.00mm_Vertical
- H1, H10, H11, H12, H13, H14, H2, H3, H4, H7, H8, H9: footprint Connector_PinHeader_1.27mm:PinHeader_1x01_P1.27mm_Vertical -> Connector_PinHeader_1.00mm:PinHeader_1x01_P1.00mm_Vertical
- R1, R2: footprint Resistor_SMD:R_0201_0603Metric -> Resistor_SMD:R_0805_2012Metric
- moved H4 10.2 mm to (73.6, 76.2)
- moved H1 5.12 mm to (66.0, 76.2)
- moved H2 2.80 mm to (71.0, 76.2)
- moved H3 2.80 mm to (68.5, 76.2)
- moved C1 2.56 mm to (61.0, 82.5)
- moved R2 1.34 mm to (73.7, 83.9)
- moved R1 1.34 mm to (67.7, 80.1)
- moved U1 1.34 mm to (67.4, 84.5)
Routing:
- net GND: track 81.0 -> 63.3 mm
- net Net-(J1-Pin_5): track 39.7 -> 53.7 mm
- net +12V: track 45.9 -> 32.8 mm, vias 2 -> 0
- net Net-(JP1-B): track 17.8 -> 7.67 mm
- net +3V3: track 22.1 -> 16.7 mm, vias 1 -> 0
- net Net-(J1-Pin_1): track 27.5 -> 22.9 mm
- net Net-(H1-Pad1): track 17.0 -> 13.0 mm
- net Net-(J1-Pin_4): track 40.1 -> 37.6 mm
- net Net-(U1-D): track 6.44 -> 8.35 mm
- net Net-(U1-R): track 6.91 -> 8.28 mm
- net Net-(U1-Rs): track 4.91 -> 4.09 mm
Other:
- board text added: "v2"
